Commit message: Move towards a working version of the package
- Right now tested just in simulation without Marrtino

File: urdf/assemblies/ur5_with_gripper.urdf.xacro (robot description, xacro)
@@ -8,7 +8,7 @@
   <xacro:include filename="$(find ur_description)/urdf/common.gazebo.xacro" />
   <!-- ur10 -->
-  <xacro:include filename="$(find ur_description)/urdf/ur5.urdf.xacro" />
+  <xacro:include filename="$(find ar_arena)/urdf/robots/ur/ur5.urdf.xacro" />
   <!-- adaptor -->
-  <xacro:include filename="$(find ar_arena)/urdf/adaptor.urdf.xacro" />
+  <xacro:include filename="$(find ar_arena)/urdf/assets/adaptor.urdf.xacro" />
   <!-- gripper -->
   <xacro:include filename="$(find robotiq_3f_gripper_visualization)/cfg/robotiq_hand_macro.urdf.xacro" />

File: urdf/assets/kinect.urdf.xacro (robot description, xacro)
@@ -1,5 +1,5 @@
 <?xml version="1.0"?>
 <root name="sensor_kinect" xmlns:xacro="http://ros.org/wiki/xacro">
-	<xacro:include filename="$(find ar_arena)/urdf/kinect2.gazebo.xacro" />
+	<xacro:include filename="$(find ar_arena)/urdf/assets/kinect2.gazebo.xacro" />
 	<xacro:include filename="$(find common_sensors)/urdf/sensors/kinect_properties.urdf.xacro"/>
    	<!-- camera_name has to be unique! -->

File: urdf/manipulator_arena_setup.urdf.xacro (robot description, xacro)
@@ -5,9 +5,9 @@
   xmlns:xacro="http://playerstage.sourceforge.net/gazebo/xmlschema/#interface"
   name="ar_ur5" >
-  <xacro:include filename="$(find ar_arena)/urdf/wall.urdf.xacro" />
-  <xacro:include filename="$(find ar_arena)/urdf/table.urdf.xacro" />
-  <xacro:include filename="$(find ar_arena)/urdf/ur_stand.urdf.xacro" />
-  <xacro:include filename="$(find ar_arena)/urdf/ur5_with_gripper.urdf.xacro" />
-  <xacro:include filename="$(find ar_arena)/urdf/kinect.urdf.xacro" />
+  <xacro:include filename="$(find ar_arena)/urdf/assets/wall.urdf.xacro" />
+  <xacro:include filename="$(find ar_arena)/urdf/assets/table.urdf.xacro" />
+  <xacro:include filename="$(find ar_arena)/urdf/assets/ur_stand.urdf.xacro" />
+  <xacro:include filename="$(find ar_arena)/urdf/assets/kinect.urdf.xacro" />
+  <xacro:include filename="$(find ar_arena)/urdf/assemblies/ur5_with_gripper.urdf.xacro" />
   <!-- setup empty world -->
   <link name="world"/>
@@ -34,15 +34,17 @@
   </joint>
   <!-- table - robot - adaptor - magnet -->
-  <xacro:ur5_with_gripper prefix="" parent="ur_stand_link" joint_limited="true">
+  <xacro:ur5_with_gripper prefix=""
+                          parent="ur_stand_link"
+                          joint_limited="$(arg joint_limited)">
     <origin xyz="0 0 0.435" rpy="0 0 0"/>
   </xacro:ur5_with_gripper>
-<!-- attach the kinect support to the table-->
-<joint name="kinect_joint" type="fixed">
-  <parent link="world" />
-  <child link = "kinect_support" />
-  <origin xyz="-0.2 -0.765 2.85" rpy="0 1.2 1.57" />
-</joint>
-<!-- kinect support-->
-<link name="kinect_support" />
+  <!-- attach the kinect support to the table-->
+  <joint name="kinect_joint" type="fixed">
+    <parent link="world" />
+    <child link = "kinect_support" />
+    <origin xyz="-0.2 -0.765 2.85" rpy="0 1.2 1.57" />
+  </joint>
+  <!-- kinect support-->
+  <link name="kinect_support" />
   <!-- add the kinect-->
   <xacro:sensor_kinect parent="kinect_support"/>

Commit message: Update robin repo

File: urdf/assemblies/ur5_with_gripper.urdf.xacro (robot description, xacro)
@@ -8,7 +8,7 @@
   <xacro:include filename="$(find ur_description)/urdf/common.gazebo.xacro" />
   <!-- ur10 -->
-  <xacro:include filename="$(find ar_arena)/urdf/robots/ur/ur5.urdf.xacro" />
+  <xacro:include filename="$(find robin_arena)/urdf/robots/ur/ur5.urdf.xacro" />
   <!-- adaptor -->
-  <xacro:include filename="$(find ar_arena)/urdf/assets/adaptor.urdf.xacro" />
+  <xacro:include filename="$(find robin_arena)/urdf/assets/adaptor.urdf.xacro" />
   <!-- gripper -->
   <xacro:include filename="$(find robotiq_3f_gripper_visualization)/cfg/robotiq_hand_macro.urdf.xacro" />

File: urdf/assemblies/ur5_with_magnet.urdf.xacro (robot description, xacro)
@@ -4,11 +4,11 @@
        xmlns:interface="http://playerstage.sourceforge.net/gazebo/xmlschema/#interface"
        xmlns:xacro="http://playerstage.sourceforge.net/gazebo/xmlschema/#interface"
-       name="ur5_no_gripper" >
+       name="ur5_with_magnet" >
   <!-- common stuff -->
   <xacro:include filename="$(find ur_description)/urdf/common.gazebo.xacro" />
   <!-- ur10 -->
-  <xacro:include filename="$(find ar_arena)/urdf/robots/ur/ur5.urdf.xacro" />
+  <xacro:include filename="$(find robin_arena)/urdf/robots/ur/ur5.urdf.xacro" />
   <!-- macro definition for ur5 robot with adaptor as a gripper -->
-  <xacro:macro name="ur5_no_gripper" params="prefix parent joint_limited *origin">
+  <xacro:macro name="ur5_with_magnet" params="prefix parent joint_limited *origin">
     <joint name="${prefix}base_joint" type="fixed">
       <parent link="${parent}"/>

File: urdf/assets/adaptor.urdf.xacro (robot description, xacro)
@@ -4,5 +4,5 @@
   xmlns:interface="http://playerstage.sourceforge.net/gazebo/xmlschema/#interface"
   xmlns:xacro="http://playerstage.sourceforge.net/gazebo/xmlschema/#interface"
-  name="ar_tool" >
+  name="robin_tool" >
   <xacro:macro name="adaptor" params="parent prefix *origin">
     <!-- mount the tool to the robot -->
@@ -21,5 +21,5 @@
         <origin xyz="0 0 0" rpy="0 0 0" />
         <geometry>
-          <mesh filename="package://ar_arena/meshes/support.dae"/>
+          <mesh filename="package://robin_arena/meshes/support.dae"/>
         </geometry>
         <material name="greyish">
@@ -30,5 +30,5 @@
         <origin xyz="0 0 0" rpy="0 0 0" />
         <geometry>
-          <mesh filename="package://ar_arena/meshes/support.dae"/>
+          <mesh filename="package://robin_arena/meshes/support.dae"/>
         </geometry>
       </collision>

File: urdf/assets/table.urdf.xacro (robot description, xacro)
@@ -1,4 +1,4 @@
 <?xml version="1.0"?>
-<robot xmlns:xacro="http://www.ros.org/wiki/xacro" name="ar_table">
+<robot xmlns:xacro="http://www.ros.org/wiki/xacro" name="robin_table">
   <xacro:macro name="table" params="">
     <static>true</static>

File: urdf/assets/ur_stand.urdf.xacro (robot description, xacro)
@@ -1,4 +1,4 @@
 <?xml version="1.0"?>
-<robot xmlns:xacro="http://www.ros.org/wiki/xacro" name="ar_ur_stand">
+<robot xmlns:xacro="http://www.ros.org/wiki/xacro" name="robin_ur_stand">
   <xacro:macro name="ur_stand" params="">
     <link name="ur_stand_link">

File: urdf/assets/wall.urdf.xacro (robot description, xacro)
@@ -1,4 +1,4 @@
 <?xml version="1.0"?>
-<robot xmlns:xacro="http://www.ros.org/wiki/xacro" name="ar_wall">
+<robot xmlns:xacro="http://www.ros.org/wiki/xacro" name="robin_wall">
   <xacro:macro name="wall" params="">
     <link name="wall_link">

File: urdf/manipulator_with_gripper_arena_setup.urdf.xacro (robot description, xacro)
@@ -4,10 +4,10 @@
   xmlns:interface="http://playerstage.sourceforge.net/gazebo/xmlschema/#interface"
   xmlns:xacro="http://playerstage.sourceforge.net/gazebo/xmlschema/#interface"
-  name="ar_ur5" >
-  <xacro:include filename="$(find ar_arena)/urdf/assets/wall.urdf.xacro" />
-  <xacro:include filename="$(find ar_arena)/urdf/assets/table.urdf.xacro" />
-  <xacro:include filename="$(find ar_arena)/urdf/assets/ur_stand.urdf.xacro" />
-  <xacro:include filename="$(find ar_arena)/urdf/assets/kinect2.urdf.xacro" />
-  <xacro:include filename="$(find ar_arena)/urdf/assemblies/ur5_no_gripper.urdf.xacro" />
+  name="robin_ur5" >
+  <xacro:include filename="$(find robin_arena)/urdf/assets/wall.urdf.xacro" />
+  <xacro:include filename="$(find robin_arena)/urdf/assets/table.urdf.xacro" />
+  <xacro:include filename="$(find robin_arena)/urdf/assets/ur_stand.urdf.xacro" />
+  <xacro:include filename="$(find robin_arena)/urdf/assets/kinect2.urdf.xacro" />
+  <xacro:include filename="$(find robin_arena)/urdf/assemblies/ur5_with_gripper.urdf.xacro" />
   <!-- setup empty world -->
   <link name="world"/>
@@ -33,10 +33,10 @@
     <origin xyz="0.0 0.0 0.435" rpy="0.0 0.0 0.0" />
   </joint>
-  <!-- table - robot - adaptor as a magnet -->
-  <xacro:ur5_no_gripper prefix=""
+  <!-- table - robot - adaptor - magnet -->
+  <xacro:ur5_with_gripper prefix=""
                           parent="ur_stand_link"
                           joint_limited="$(arg joint_limited)">
     <origin xyz="0 0 0.435" rpy="0 0 0"/>
-  </xacro:ur5_no_gripper>
+  </xacro:ur5_with_gripper>
   <!-- attach the kinect support to the table-->
   <!-- <joint name="kinect_joint" type="fixed">

File: urdf/manipulator_with_magnet_arena_setup.urdf.xacro (robot description, xacro)
@@ -4,10 +4,10 @@
   xmlns:interface="http://playerstage.sourceforge.net/gazebo/xmlschema/#interface"
   xmlns:xacro="http://playerstage.sourceforge.net/gazebo/xmlschema/#interface"
-  name="ar_ur5" >
-  <xacro:include filename="$(find ar_arena)/urdf/assets/wall.urdf.xacro" />
-  <xacro:include filename="$(find ar_arena)/urdf/assets/table.urdf.xacro" />
-  <xacro:include filename="$(find ar_arena)/urdf/assets/ur_stand.urdf.xacro" />
-  <xacro:include filename="$(find ar_arena)/urdf/assets/kinect2.urdf.xacro" />
-  <xacro:include filename="$(find ar_arena)/urdf/assemblies/ur5_with_gripper.urdf.xacro" />
+  name="robin_ur5" >
+  <xacro:include filename="$(find robin_arena)/urdf/assets/wall.urdf.xacro" />
+  <xacro:include filename="$(find robin_arena)/urdf/assets/table.urdf.xacro" />
+  <xacro:include filename="$(find robin_arena)/urdf/assets/ur_stand.urdf.xacro" />
+  <xacro:include filename="$(find robin_arena)/urdf/assets/kinect2.urdf.xacro" />
+  <xacro:include filename="$(find robin_arena)/urdf/assemblies/ur5_no_gripper.urdf.xacro" />
   <!-- setup empty world -->
   <link name="world"/>
@@ -33,10 +33,10 @@
     <origin xyz="0.0 0.0 0.435" rpy="0.0 0.0 0.0" />
   </joint>
-  <!-- table - robot - adaptor - magnet -->
-  <xacro:ur5_with_gripper prefix=""
+  <!-- table - robot - adaptor as a magnet -->
+  <xacro:ur5_no_gripper prefix=""
                           parent="ur_stand_link"
                           joint_limited="$(arg joint_limited)">
     <origin xyz="0 0 0.435" rpy="0 0 0"/>
-  </xacro:ur5_with_gripper>
+  </xacro:ur5_no_gripper>
   <!-- attach the kinect support to the table-->
   <!-- <joint name="kinect_joint" type="fixed">

File: urdf/robots/ur/ur5.urdf.xacro (robot description, xacro)
@@ -2,5 +2,5 @@
 <robot xmlns:xacro="http://wiki.ros.org/xacro">
   <xacro:include filename="$(find ur_description)/urdf/ur.transmission.xacro" />
-  <xacro:include filename="$(find ar_arena)/urdf/robots/ur/ur.gazebo.xacro" />
+  <xacro:include filename="$(find robin_arena)/urdf/robots/ur/ur.gazebo.xacro" />
   <xacro:macro name="cylinder_inertial" params="radius length mass *origin">
     <inertial>
