Commit message: Update robin repo

File: urdf/assemblies/ur5_3fgripper.urdf.xacro (robot description, xacro)
@@ -4,5 +4,5 @@
        xmlns:interface="http://playerstage.sourceforge.net/gazebo/xmlschema/#interface"
        xmlns:xacro="http://playerstage.sourceforge.net/gazebo/xmlschema/#interface"
-       name="ur5_with_gripper" >
+       name="ur5_3fgripper" >
   <!-- common stuff -->
   <xacro:include filename="$(find ur_description)/urdf/common.gazebo.xacro" />
@@ -13,6 +13,6 @@
   <!-- gripper -->
   <xacro:include filename="$(find robotiq_3f_gripper_visualization)/cfg/robotiq_hand_macro.urdf.xacro" />
-  <!-- macro definition for ur5 robot with gripper -->
-  <xacro:macro name="ur5_with_gripper" params="prefix parent joint_limited *origin">
+  <!-- macro definition for ur5 robot with 3-finger gripper -->
+  <xacro:macro name="ur5_3fgripper" params="prefix parent joint_limited *origin">
     <joint name="${prefix}base_joint" type="fixed">
       <parent link="${parent}"/>

File: urdf/assemblies/ur5_magnet.urdf.xacro (robot description, xacro)
@@ -4,11 +4,11 @@
        xmlns:interface="http://playerstage.sourceforge.net/gazebo/xmlschema/#interface"
        xmlns:xacro="http://playerstage.sourceforge.net/gazebo/xmlschema/#interface"
-       name="ur5_with_magnet" >
+       name="ur5_magnet" >
   <!-- common stuff -->
   <xacro:include filename="$(find ur_description)/urdf/common.gazebo.xacro" />
   <!-- ur10 -->
   <xacro:include filename="$(find robin_arena)/urdf/robots/ur/ur5.urdf.xacro" />
-  <!-- macro definition for ur5 robot with adaptor as a gripper -->
-  <xacro:macro name="ur5_with_magnet" params="prefix parent joint_limited *origin">
+  <!-- macro definition for ur5 robot with magnet -->
+  <xacro:macro name="ur5_magnet" params="prefix parent joint_limited *origin">
     <joint name="${prefix}base_joint" type="fixed">
       <parent link="${parent}"/>

File: urdf/manipulator_ur5_3fgripper_arena_setup.urdf.xacro (robot description, xacro)
@@ -9,5 +9,5 @@
   <xacro:include filename="$(find robin_arena)/urdf/assets/ur_stand.urdf.xacro" />
   <xacro:include filename="$(find robin_arena)/urdf/assets/kinect2.urdf.xacro" />
-  <xacro:include filename="$(find robin_arena)/urdf/assemblies/ur5_with_gripper.urdf.xacro" />
+  <xacro:include filename="$(find robin_arena)/urdf/assemblies/ur5_3fgripper.urdf.xacro" />
   <!-- setup empty world -->
   <link name="world"/>
@@ -34,9 +34,9 @@
   </joint>
   <!-- table - robot - adaptor - magnet -->
-  <xacro:ur5_with_gripper prefix=""
+  <xacro:ur5_3fgripper prefix=""
                           parent="ur_stand_link"
                           joint_limited="$(arg joint_limited)">
     <origin xyz="0 0 0.435" rpy="0 0 0"/>
-  </xacro:ur5_with_gripper>
+  </xacro:ur5_3fgripper>
   <!-- attach the kinect support to the table-->
   <!-- <joint name="kinect_joint" type="fixed">
